File: _autosave-babySwerveController.kicad_sch (KiCad schematic)
At the start: 34 parts, among them J1 Conn_01x07_Female, J2 pgm, J3 Conn_01x06_Male, J4 Conn_01x06_Male, J5 USB_B_Micro, SW1 sw, U1 ATmega32U4-A, U2 MT1470, U3 TLV75533PDBV, U6 TB6612FNG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

Commit message: Atmega32u4 rev
Other:
- note added: "CONTROL"
- note added: "INTERFACING"
- note added: "MOTOR CONTROL"
- note added: "POWER"
- moved on the sheet: C10, C11, C12, C3, C6, C7, C8, C9, H1, H2, L1, R5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
