File: babySwerveController.kicad_pcb (KiCad board)
At the start: 2 copper layers, 35.6 x 24.8 mm, 20 parts, among them J1 interBoardConnect, J2 pgm, J3 Conn_01x06_Male, J4 Conn_01x06_Male, SW1 sw, U1 LF18_TO252, U2 LF33_TO252, U3 STM32F038G6Ux, U4 TXB0104RUT, U5 TXB0104RUT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

Commit message: Atmega32u4 rev
Parts:
- removed U4, U5: TXB0104RUT, Package_DFN_QFN:Texas_R_PUQFN-N12
- added C10: 1uF, Capacitor_SMD:C_0603_1608Metric, F.Cu at (93.6, 139.7)
- added C11: 1uF, Capacitor_SMD:C_0603_1608Metric, F.Cu at (92.8, 133.9)
- added C12: 10uF, Capacitor_SMD:C_0603_1608Metric, F.Cu at (99.7, 121.1)
- added C6: 1uF, Capacitor_SMD:C_0402_1005Metric, F.Cu at (230.7, 106.1)
- added C7: 22uF, Capacitor_SMD:C_0402_1005Metric, F.Cu at (231.5, 104.3)
- added C8: 22uF, Capacitor_SMD:C_0402_1005Metric, F.Cu at (232.8, 101.4)
- added C9: 22uF, Capacitor_SMD:C_0402_1005Metric, F.Cu at (229.9, 97.8)
- added J5: USB_B_Micro, Connector_USB:USB_Micro-B_Amphenol_10118194_Horizontal, F.Cu at (89.4, 119.7)
- added L1: 11uH, Inductor_SMD:L_10.4x10.4_H4.8, F.Cu at (221.4, 100.8)
- added R2: 22, Resistor_SMD:R_0402_1005Metric, F.Cu at (92.2, 123.7)
- added R3: 22, Resistor_SMD:R_0402_1005Metric, F.Cu at (93.4, 123.7)
- added R4: 10k, Resistor_SMD:R_0603_1608Metric, F.Cu at (104.0, 121.2)
- added R5: 200k, Resistor_SMD:R_0201_0603Metric, F.Cu at (235.2, 95.9)
- added R6: 100k, Resistor_SMD:R_0201_0603Metric, F.Cu at (231.1, 100.0)
- added R7: 18.7k, Resistor_SMD:R_0201_0603Metric, F.Cu at (234.2, 97.5)
- added Y1: Crystal, Crystal:Crystal_SMD_TXC_7M-4Pin_3.2x2.5mm, F.Cu at (100.4, 138.9)
- C1: value 100nF -> 1uF
- C2: value 100nF -> 22pF; footprint Capacitor_SMD:C_0603_1608Metric -> Capacitor_SMD:C_0402_1005Metric
- C3: value 10nF -> 10uF
- C4: value 4.7uF -> 1uF
- C5: value 0.1uF -> 22pF; footprint Capacitor_SMD:C_0201_0603Metric -> Capacitor_SMD:C_0402_1005Metric
- J1: value interBoardConnect -> Conn_01x07_Female; footprint Connector_PinSocket_2.54mm:PinSocket_1x06_P2.54mm_Vertical -> Connector_PinHeader_2.54mm:PinHeader_1x07_P2.54mm_Horizontal
- JP1: value bootJumper -> Jumper; footprint Connector_PinHeader_1.00mm:PinHeader_1x02_P1.00mm_Vertical -> Connector_PinHeader_2.54mm:PinHeader_1x03_P2.54mm_Vertical
- U1: value LF18_TO252 -> ATmega32U4-A; footprint Package_TO_SOT_SMD:TO-252-2 -> Package_QFP:TQFP-44_10x10mm_P0.8mm
- U2: value LF33_TO252 -> MT1470; footprint Package_TO_SOT_SMD:TO-252-2 -> Package_TO_SOT_SMD:SOT-23-6
- U3: value STM32F038G6Ux -> TLV75533PDBV; footprint Package_DFN_QFN:QFN-28_4x4mm_P0.5mm -> Package_TO_SOT_SMD:SOT-23-5
- moved U2 111.4 mm to (220.9, 109.4)
- moved H2 23.6 mm to (127.6, 120.1)
- moved J1 23.6 mm to (89.8, 139.7), turned to 180 degrees
- moved C2 18.3 mm to (103.2, 138.1), turned to 90 degrees
- moved U3 16.1 mm to (94.2, 137.3), turned to 0 degrees
- moved C5 12.2 mm to (97.6, 138.1), turned to -90 degrees
- moved R1 12.0 mm to (105.9, 137.2)
- moved C3 8.82 mm to (108.4, 135.3)
- moved H1 8.26 mm to (127.6, 137.9)
- moved JP1 8.21 mm to (96.5, 118.5), turned to 90 degrees
- moved C1 7.83 mm to (96.2, 121.2)
- moved SW1 7.69 mm to (111.1, 135.2), turned to -90 degrees
- moved C4 7.05 mm to (92.6, 127.7), turned to 90 degrees
- moved J3 5.59 mm to (121.4, 133.6)
- moved J4 5.59 mm to (121.4, 123.6)
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Connections:
- C1 pad 1: +1V8 -> +5V
- C2 pad 1: +1V8 -> GND
- C2 pad 2: GND -> Net-(C2-Pad2)
- C3 pad 1: +1V8 -> +3.3V
- C4 pad 1: +1V8 -> Net-(C4-Pad1)
- C5 pad 1: GND -> Net-(C5-Pad1)
- C5 pad 2: Net-(C5-Pad2) -> GND
- J1 pad 1: GND -> /VBATT
- J1 pad 2: /SPI_SCLK -> +5V
- J1 pad 5: /SPI_NSS -> /SPI_SCLK
- J1 pad 6: /VBATT -> /SPI_NSS
- J2 pad 2: /UART_TX -> /UART_RX
- J2 pad 3: /UART_RX -> /UART_TX
- J4 pad 3: /qEncoderA2 -> /UART_TX
- J4 pad 4: /qEncoderB2 -> /UART_RX
- JP1 pad 1: +3.3V -> GND
- R1 pad 1: GND -> Net-(R1-Pad1)
- R1 pad 2: Net-(JP1-Pad2) -> +3.3V
- SW1 pad 1: Net-(C5-Pad2) -> Net-(R1-Pad1)
- U1 pad 1: /VBATT -> unconnected-(U1-Pad1)
- U1 pad 2: GND -> +5V
- U1 pad 3: +1V8 -> Net-(R3-Pad2)
- U2 pad 1: /VBATT -> GND
- U2 pad 2: GND -> Net-(C6-Pad1)
- U2 pad 3: +3.3V -> /VBATT
- U3 pad 1: Net-(JP1-Pad2) -> +5V
- U3 pad 2: unconnected-(U3-Pad2) -> GND
- U3 pad 3: unconnected-(U3-Pad3) -> +5V
- U3 pad 4: Net-(C5-Pad2) -> unconnected-(U3-Pad4)
- U3 pad 5: +1V8 -> +3.3V
Routing:
- net +1V8: track 49.1 -> 0.00 mm, vias 10 -> 0
- net +5V: track 0.00 -> 34.8 mm
- net /qEncoderB2: track 30.0 -> 0.00 mm, vias 2 -> 0
- net /qEncoderA2: track 26.2 -> 0.00 mm, vias 2 -> 0
- net Net-(R1-Pad1): track 0.00 -> 24.3 mm, vias 0 -> 2
- net /UART_RX: track 17.8 -> 40.7 mm, vias 1 -> 2
- net /VBATT: track 24.4 -> 47.1 mm, vias 16 -> 4
- net /STBY_1V8: track 14.0 -> 0.00 mm
- net /AIN2: track 3.35 -> 16.8 mm, vias 0 -> 2
- net /AIN1: track 3.45 -> 14.2 mm, vias 0 -> 2
- net Net-(C5-Pad2): track 9.63 -> 0.00 mm
- net /PWM2H_1V8: track 8.45 -> 0.00 mm, vias 2 -> 0
- net /BIN2: track 3.74 -> 11.3 mm, vias 0 -> 2
- net /UART_TX: track 23.4 -> 30.9 mm, vias 1 -> 2
- net /BIN1: track 4.98 -> 12.2 mm
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- removed copper zone on B.Cu, net /VBATT
Other:
- board size 35.6 x 24.8 mm -> 46.6 x 24 mm
